Commit message: Updated rmp_2023

File: rmp_2023/urdf/controller.gazebo.xacro (robot description, xacro)
@@ -25,5 +25,5 @@
       <odometryFrame>odom</odometryFrame>
       <odometryRate>100.0</odometryRate>
-      <robotBaseFrame>base_link</robotBaseFrame>
+      <robotBaseFrame>base_dummy</robotBaseFrame>
       <publishTF>true</publishTF>
     </plugin>

File: rmp_2023/urdf/lidar.gazebo.xacro (robot description, xacro)
@@ -6,5 +6,5 @@
         <!--<sensor name='sensor' type='gpu_ray'> -->
           <!-- <pose frame=''>0.0 0.0 0.5 0.0 0.0 0.0</pose> -->
-          <visualize>0</visualize>
+          <visualize>1</visualize>
           <update_rate>50</update_rate>
           <ray>
@@ -23,5 +23,5 @@
             </scan>
             <range>
-              <min>0.05</min>
+              <min>0.1</min>
               <max>10</max>
               <resolution>0.02</resolution>

File: rmp_2023/urdf/robot_base.urdf.xacro (robot description, xacro)
@@ -2,4 +2,10 @@
 <robot name="pioneer" xmlns:xacro="http://www.ros.org/wiki/xacro">
   <xacro:macro name="robot_base">
+  <gazebo reference="castor_wheel_link">
+    <material>Gazebo/Black</material>
+  </gazebo>
+  <gazebo reference="lidar_link">
+    <material>Gazebo/Black</material>
+  </gazebo>
   <!-- Dummy link -->
   <link name="base_dummy">
@@ -11,4 +17,5 @@
     </visual>
   </link>
+  <!-- BASE LINK  -->
   <link name="base_link">
     <inertial>
@@ -19,5 +26,5 @@
       <origin rpy="0 0 0" xyz="0 0 0"/>
       <geometry>
-        <mesh filename="model://pioneer2dx/model.sdf"/>
+        <mesh filename="model://pioneer2dx/meshes/chassis.dae"/>
       </geometry>
     </visual>
@@ -25,5 +32,5 @@
       <origin xyz="0 0 0" rpy="0 0 0" />
       <geometry>
-        <mesh filename="model://pioneer2dx/model.sdf"/>
+        <mesh filename="model://pioneer2dx/meshes/chassis.dae"/>
       </geometry>
     </collision>
@@ -34,9 +41,79 @@
       <child link="base_link" />
   </joint>
+  <!-- WHEELS  -->
+  <link name="left_wheel_link">
+    <inertial>
+      <mass value="0.1"/>
+      <inertia ixx="0.0407" ixy="0.0" ixz="0.0" iyy="0.0407" iyz="0.0" izz="0.0756"/>
+    </inertial>
+    <visual>
+      <origin rpy="0 0 0" xyz="0 0 0"/>
+      <geometry>
+        <mesh filename="model://pioneer2dx/meshes/wheel.dae"/>
+      </geometry>
+    </visual>
+    <collision>
+      <origin xyz="0 0 0" rpy="0 0 0" />
+      <geometry>
+        <mesh filename="model://pioneer2dx/meshes/wheel.dae"/>
+      </geometry>
+    </collision>
+  </link>
+  <joint name="left_wheel_joint" type="fixed">
+      <origin xyz="0.1 .17 -0.09" rpy="0 1.5707 0" />
+      <parent link="base_link"/>
+      <child link="left_wheel_link" />
+  </joint>
+  <link name="right_wheel_link">
+    <inertial>
+      <mass value="0.1"/>
+      <inertia ixx="0.0407" ixy="0.0" ixz="0.0" iyy="0.0407" iyz="0.0" izz="0.0756"/>
+    </inertial>
+    <visual>
+      <origin rpy="0 0 0" xyz="0 0 0"/>
+      <geometry>
+        <mesh filename="model://pioneer2dx/meshes/wheel.dae"/>
+      </geometry>
+    </visual>
+    <collision>
+      <origin xyz="0 0 0" rpy="0 0 0" />
+      <geometry>
+        <mesh filename="model://pioneer2dx/meshes/wheel.dae"/>
+      </geometry>
+    </collision>
+  </link>
+  <joint name="right_wheel_joint" type="fixed">
+      <origin xyz="0.1 -.17 -0.09" rpy="0 1.5707 3.1415" />
+      <parent link="base_link"/>
+      <child link="right_wheel_link" />
+  </joint>
+  <link name="castor_wheel_link">
+    <visual>
+      <origin rpy="0 0 0" xyz="0 0 0"/>
+      <geometry>
+        <sphere radius="0.04"/>
+      </geometry>
+      <material name="black">
+            <color rgba="1 1 1 1"/>
+      </material>
+    </visual>
+    <collision>
+      <origin xyz="0 0 0" rpy="0 0 0" />
+      <geometry>
+        <sphere radius="0.04"/>
+      </geometry>
+    </collision>
+  </link>
+  <joint name="castor_wheel_joint" type="fixed">
+      <origin xyz="-0.200 0 -0.16" rpy="0 0 0" />
+      <parent link="base_link"/>
+      <child link="castor_wheel_link" />
+  </joint>
+  <!-- LIDAR -->
   <link name="lidar_link">
     <visual>
-      <pose xyz="0 0 0.3"/>
+      <pose xyz="0 0 0"/>
       <geometry>
-        <box size="0.001 0.001 0.001" />
+        <cylinder length="0.05" radius="0.049"/>
       </geometry>
     </visual>
@@ -45,5 +122,5 @@
     <parent link="base_link"/>
     <child link="lidar_link"/>
-    <origin xyz="0 0 0.3"/>
+    <origin xyz="0 0 0.085"/>
   </joint>
   </xacro:macro>

Commit message: Add files via upload

File: rmp_2023/urdf/controller.gazebo.xacro (robot description, xacro)
@@ -2,22 +2,30 @@
 <robot xmlns:xacro="http://www.ros.org/wiki/xacro">
 <xacro:macro name="controller" params="">
-	<!--
+<!--        <gazebo>
+          <plugin name="gazebo_ros_control" filename="libgazebo_ros_control.so">
+          </plugin>
+        </gazebo>
+-->
 	<gazebo>
 	  <plugin name="differential_drive_controller" filename="libgazebo_ros_diff_drive.so">
 	    <alwaysOn>true</alwaysOn>
-	    <updateRate>60</updateRate>
-	    <leftJoint>right_wheel_joint</leftJoint>
-	    <rightJoint>left_wheel_joint</rightJoint>
-	    <wheelSeparation>0.275</wheelSeparation>
+	    <updateRate>40</updateRate>
+	    <leftJoint>left_wheel_joint</leftJoint>
+	    <rightJoint>right_wheel_joint</rightJoint>
+	    <wheelSeparation>0.17</wheelSeparation>
 	    <wheelDiameter>0.1</wheelDiameter>
-	    <torque>20</torque>
 	    <commandTopic>cmd_vel</commandTopic>
 	    <odometryTopic>odom</odometryTopic>
 	    <odometryFrame>odom</odometryFrame>
 	    <robotBaseFrame>base_link</robotBaseFrame>
+            <publishOdom>false</publishOdom>
+            <publishOdomTF>false</publishOdomTF>
+            <legacyMode>false</legacyMode>
+            <!-- <odometrySource>1</odometrySource> -->
+            <wheelTorque>5</wheelTorque>
 	  </plugin>
 	</gazebo>
-	-->
-	<gazebo>
+  <!--
+  <gazebo>
     <plugin name="omni_steering" filename="libgazebo_ros_planar_move.so">
       <commandTopic>cmd_vel</commandTopic>
@@ -25,8 +33,8 @@
       <odometryFrame>odom</odometryFrame>
       <odometryRate>100.0</odometryRate>
-      <robotBaseFrame>base_dummy</robotBaseFrame>
-      <publishTF>true</publishTF>
+      <robotBaseFrame>base_link</robotBaseFrame>
+      <publishTF>0</publishTF>
     </plugin>
-  </gazebo>
+  </gazebo> -->
 </xacro:macro>
 </robot>

File: rmp_2023/urdf/lidar.gazebo.xacro (robot description, xacro)
@@ -11,8 +11,10 @@
             <scan>
               <horizontal>
-                <samples>400</samples>
+                <samples>200</samples>
                 <resolution>1</resolution>
-                <min_angle>0</min_angle>
-                <max_angle>6.2832</max_angle>
+                <!-- <min_angle>0</min_angle>
+                <max_angle>6.2832</max_angle> -->
+                <min_angle>-1.5707</min_angle>
+                <max_angle>1.5707</max_angle>
               </horizontal>
               <vertical>
@@ -24,5 +26,5 @@
             <range>
               <min>0.1</min>
-              <max>10</max>
+              <max>6</max>
               <resolution>0.02</resolution>
             </range>

File: rmp_2023/urdf/robot_base.urdf.xacro (robot description, xacro)
@@ -2,4 +2,5 @@
 <robot name="pioneer" xmlns:xacro="http://www.ros.org/wiki/xacro">
   <xacro:macro name="robot_base">
+  <!--############################ MATERIAL DEFINITION ##########################-->
   <gazebo reference="castor_wheel_link">
     <material>Gazebo/Black</material>
@@ -8,5 +9,5 @@
     <material>Gazebo/Black</material>
   </gazebo>
-  <!-- Dummy link -->
+  <!--############################ DUMMY LINK ##########################-->
   <link name="base_dummy">
     <visual>
@@ -17,9 +18,9 @@
     </visual>
   </link>
-  <!-- BASE LINK  -->
+  <!--############################ BASE LINK ##########################-->
   <link name="base_link">
     <inertial>
-      <mass value="2"/>
-      <inertia ixx="0.0407" ixy="0.0" ixz="0.0" iyy="0.0407" iyz="0.0" izz="0.0756"/>
+      <mass value="5.67" />
+      <inertia ixx="0.07" ixy="0.0" ixz="0.0" iyy="0.08" iyz="0.0" izz="0.10" />
     </inertial>
     <visual>
@@ -41,9 +42,9 @@
       <child link="base_link" />
   </joint>
-  <!-- WHEELS  -->
+  <!--############################ LEFT WHEEL ##########################-->
   <link name="left_wheel_link">
     <inertial>
-      <mass value="0.1"/>
-      <inertia ixx="0.0407" ixy="0.0" ixz="0.0" iyy="0.0407" iyz="0.0" izz="0.0756"/>
+      <mass value="1.5" />
+      <inertia ixx="0.0051" ixy="0.0" ixz="0.0" iyy="0.0051" iyz="0.0" izz="0.0090" />
     </inertial>
     <visual>
@@ -58,18 +59,30 @@
         <mesh filename="model://pioneer2dx/meshes/wheel.dae"/>
       </geometry>
+      <surface>
+          <friction>
+            <ode>
+              <mu>100000.0</mu>
+              <mu2>100000.0</mu2>
+              <slip1>0.0</slip1>
+              <slip2>0.0</slip2>
+            </ode>
+          </friction>
+        </surface>
     </collision>
   </link>
-  <joint name="left_wheel_joint" type="fixed">
+  <joint name="left_wheel_joint" type="continuous">
       <origin xyz="0.1 .17 -0.09" rpy="0 1.5707 0" />
       <parent link="base_link"/>
       <child link="left_wheel_link" />
+      <axis xyz="0 1 0" />
   </joint>
+  <!--############################ RIGHT WHEEL ##########################-->
   <link name="right_wheel_link">
     <inertial>
-      <mass value="0.1"/>
-      <inertia ixx="0.0407" ixy="0.0" ixz="0.0" iyy="0.0407" iyz="0.0" izz="0.0756"/>
+      <mass value="1.5" />
+      <inertia ixx="0.0051" ixy="0.0" ixz="0.0" iyy="0.0051" iyz="0.0" izz="0.0090" />
     </inertial>
     <visual>
-      <origin rpy="0 0 0" xyz="0 0 0"/>
+      <origin rpy="0 0 3.1415" xyz="0 0 0"/>
       <geometry>
         <mesh filename="model://pioneer2dx/meshes/wheel.dae"/>
@@ -81,11 +94,23 @@
         <mesh filename="model://pioneer2dx/meshes/wheel.dae"/>
       </geometry>
+      <surface>
+          <friction>
+            <ode>
+              <mu>100000.0</mu>
+              <mu2>100000.0</mu2>
+              <slip1>0.0</slip1>
+              <slip2>0.0</slip2>
+            </ode>
+          </friction>
+        </surface>
     </collision>
   </link>
-  <joint name="right_wheel_joint" type="fixed">
-      <origin xyz="0.1 -.17 -0.09" rpy="0 1.5707 3.1415" />
+  <joint name="right_wheel_joint" type="continuous">
+      <origin xyz="0.1 -.17 -0.09" rpy="0 1.5707 0" />
       <parent link="base_link"/>
       <child link="right_wheel_link" />
+      <axis xyz="0 1 0" />
   </joint>
+  <!--############################ CASTOR WHEEL ##########################-->
   <link name="castor_wheel_link">
     <visual>
@@ -103,4 +128,14 @@
         <sphere radius="0.04"/>
       </geometry>
+      <surface>
+          <friction>
+            <ode>
+              <mu>0</mu>
+              <mu2>0</mu2>
+              <slip1>1.0</slip1>
+              <slip2>1.0</slip2>
+            </ode>
+          </friction>
+        </surface>
     </collision>
   </link>
@@ -110,5 +145,5 @@
       <child link="castor_wheel_link" />
   </joint>
-  <!-- LIDAR -->
+  <!--############################ LIDAR LINK ##########################-->
   <link name="lidar_link">
     <visual>
